File: hardware/buffer_overflow.kicad_sch (KiCad schematic)
At the start: 21 parts, among them J2 E1, J2 UX1, J3 UX2, U1 LM741

Commit message: Fix issue detected in hardware version v0.40
 - swap backwards volume knob pins
Connections:
- net GND: now also J2.25 (Pin_25); no longer J2.23 (Pin_23)
- net POT3_CCW renamed POT3_CW
- net POT3_CW: now also J2.23 (Pin_23); no longer J2.25 (Pin_25)
